File: PCB/TFG53/tfg53.kicad_pcb (KiCad board)
At the start: 2 copper layers, 190 x 90 mm, 31 parts, among them J2 N, J4 Thermocuple, J5 L, J6 Iin, J7 Iout, J8 IN, Q1 BTA16-600B, U1 ESP32-DEVKIT-V1, U2 HS96L03W2C03, U3 PC817, U4 MOC3010

Commit message: Gerber files
Parts:
- added G***: LOGO, logo:logo16x16mm, F.Cu at (86.4, 61.2)
- renumbered R7 to 100, R5 to 1K, R2 to 1K, R1 to 1K, R6 to 220, R3 to 47K, R4 to 47K, Q1 to BTA, PS1 to HLK-PM01, R8 to Heater, J7 to INL, J8 to INN, J6 to INTEPT, D1 to KBPC610, U4 to MOC3010, U2 to OLED, U3 to PC817, J4 to TK, J5 to VIL, J2 to VIN
Routing:
- net SO: track 54.9 -> 57.8 mm, vias 0 -> 1
- net Net-(D1-Pad2): track 18.4 -> 17.3 mm
- net SDA: track 61.3 -> 61.4 mm, vias 0 -> 1
Other:
- board text added: "ThermoForge TFG-ET V1"
