File: PCB/TFG53/tfg53.kicad_sch (KiCad schematic)
At the start: 33 parts, among them J1 Conn_02x01, J11 12V, J2 LCD, J3 Conn_02x01, J4 Conn_02x01, J5 AC TO HEATER, J6 120V, J7 AC SUPPLY, J8 Conn_02x01, J9 TERMO K, U1 ESP32-DEVKIT-V1, U2 AMS1117, U3 INA128P, U4 LM35CAZ/NOPB

Commit message: Optoacoplador MOC3010 added
Parts:
- added U5: MOC3010, TFGMOC:DIP-6_L9.6-W6.4-P2.54-LS7.6-BL, symbol TFGMOC:MOC3010
Changed lines of the file:
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@@
+    )
+  )
+  (symbol (lib_id "TFGMOC:MOC3010") (at 200.66 127 0) (unit 1)
+    (in_bom yes) (on_board yes) (dnp no) (fields_autoplaced)
+    (property "Reference" "U5" (at 200.66 116.84 0)
+      (effects (font (size 1.27 1.27)))
+    )
+    (property "Value" "MOC3010" (at 200.66 119.38 0)
+      (effects (font (size 1.27 1.27)))
+    )
+    (property "Footprint" "TFGMOC:DIP-6_L9.6-W6.4-P2.54-LS7.6-BL" (at 200.66 139.7 0)
+      (effects (font (size 1.27 1.27)) hide)
+    )
+    (property "Datasheet" "https://wmsc.lcsc.com/wmsc/upload/file/pdf/v2/lcsc/2402291825_Texas-Instruments-MOC3010_C6595293.pdf" (at 200.66 127 0)
+      (effects (font (size 1.27 1.27)) hide)
+    )
+    (property "LCSC Part" "C6595293" (at 200.66 142.24 0)
+      (effects (font (size 1.27 1.27)) hide)
+    )
+    (pin "1")
+    (pin "2")
+    (pin "3")
+    (pin "4")
+    (pin "5")
+    (pin "6")
+    (instances
+      (project "tfg53"
+        (path "/4a9374d1-a52e-4006-9aab-30b6556280a8"
+          (reference "U5") (unit 1)
+        )
+      )
     )
   )

Commit message: Termocuple code
Parts:
- removed C1: 10nF, Capacitor_SMD:C_1206_3216Metric, symbol Device:C
- removed C2: 100uF, Capacitor_SMD:CP_Elec_6.3x7.7, symbol Device:C_Polarized_US
- removed C3: 10uF, Capacitor_SMD:CP_Elec_6.3x7.7, symbol Device:C_Polarized_US
- removed D1, D2, D3, D4: 1N4001, digikey-footprints:DO-214AC, symbol Diode:1N4001
- removed J11: 12V, TerminalBlock_4Ucon:TerminalBlock_4Ucon_1x02_P3.50mm_Horizontal, symbol Connector:Screw_Terminal_01x02
- removed J6: 120V, TerminalBlock_4Ucon:TerminalBlock_4Ucon_1x02_P3.50mm_Horizontal, symbol Connector:Screw_Terminal_01x02
- removed U2: AMS1117, Package_TO_SOT_SMD:SOT-223-3_TabPin2, symbol Regulator_Linear:AMS1117
- added D5: KBPC606, easyeda2kicad:DIO-BG-TH_KBPC6, symbol TFGKBPC:KBPC606
- added R7: 22k, Resistor_SMD:R_1206_3216Metric, symbol Device:R
- added R9: 100k, Resistor_SMD:R_1206_3216Metric, symbol Device:R
- added U6: HLK-PM01, TFGHLK:PWRM-TH_HLK-PM01, symbol TFGHLK:HLK-PM01
- R1: value 220 -> 10K
- R2, R3, R4: value 220 -> 10k
Connections:
- net +5V: now also R9.2, U6.4 (+VO)
- net AC A: now also D5.2 (AC), U6.1 (AC)
- net AC B: now also D5.4 (AC), U6.2 (AC)
- net GND: now also U5.4, U6.3 (-VO)
- net at U5.1: now also R7.1
- net at U5.2: now also D5.3 (-)
- net at U5.6: now also R9.1
- new net: D5.1 (+), R7.2
Other:
- note added: "FEEDBACK"
- note removed: "RETROALIMENTATION"
- note removed: "TRANSFORMER"
- moved on the sheet: U5

Commit message: Placa terminada
Parts:
- removed D5: KBPC606, easyeda2kicad:DIO-BG-TH_KBPC6, symbol TFGKBPC:KBPC606
- removed H5, H6: MountingHole, MountingHole:MountingHole_3.2mm_M3_Pad_Via, symbol Mechanical:MountingHole
- removed J1, J3, J4, J8: Conn_02x01, Button_Switch_THT:SW_PUSH_6mm_H5mm, symbol Connector_Generic:Conn_02x01
- removed J2: LCD, Connector_PinHeader_2.54mm:PinHeader_1x04_P2.54mm_Vertical, symbol Connector_Generic:Conn_01x04
- removed J5: AC TO HEATER, TerminalBlock_4Ucon:TerminalBlock_4Ucon_1x02_P3.50mm_Horizontal, symbol Connector:Screw_Terminal_01x02
- removed J7: AC SUPPLY, TerminalBlock_4Ucon:TerminalBlock_4Ucon_1x02_P3.50mm_Horizontal, symbol Connector:Screw_Terminal_01x02
- removed J9: TERMO K, TerminalBlock_4Ucon:TerminalBlock_4Ucon_1x02_P3.50mm_Horizontal, symbol Connector:Screw_Terminal_01x02
- removed R5: R_V 500, symbol Device:R_Variable
- removed R8: R_V 300, symbol Device:R_Variable
- removed R9: 100k, Resistor_SMD:R_1206_3216Metric, symbol Device:R
- removed U3: INA128P, TFGINA:PDIP-8_L9.6-W6.4-P2.54-LS7.9-BL, symbol TFGINA:INA128P
- removed U4: LM35CAZ/NOPB, TFGLM:TO-92-3_L4.8-W3.7-P1.27-L, symbol TFGLM:LM35CAZ_NOPB
- removed U5: MOC3010, TFGMOC:DIP-6_L9.6-W6.4-P2.54-LS7.6-BL, symbol TFGMOC:MOC3010
- removed U6: HLK-PM01, TFGHLK:PWRM-TH_HLK-PM01, symbol TFGHLK:HLK-PM01
- added D1: VS-KBPC610, Diode_THT:Diode_Bridge_Vishay_KBPC6, symbol Diode_Bridge:VS-KBPC610
- added F1: 16A, Fuse:Fuseholder_Cylinder-5x20mm_Stelvio-Kontek_PTF78_Horizontal_Open, symbol Device:Fuse
- added F3: 1A, Fuse:Fuseholder_Cylinder-5x20mm_Stelvio-Kontek_PTF78_Horizontal_Open, symbol Device:Fuse
- added H1, H2: MH, MountingHole:MountingHole_3mm_Pad_Via, symbol Mechanical:MountingHole
- added J2: N, TerminalBlock_MetzConnect:TerminalBlock_MetzConnect_360271_1x01_Horizontal_ScrewM3.0_Boxed, symbol Connector:Screw_Terminal_01x01
- added J4: Thermocuple, Connector_PinHeader_2.54mm:PinHeader_1x05_P2.54mm_Vertical, symbol Connector:Conn_01x05_Pin
- added J5: L, TerminalBlock_MetzConnect:TerminalBlock_MetzConnect_360271_1x01_Horizontal_ScrewM3.0_Boxed, symbol Connector:Screw_Terminal_01x01
- added J6: Iin, TerminalBlock_MetzConnect:TerminalBlock_MetzConnect_360271_1x01_Horizontal_ScrewM3.0_Boxed, symbol Connector:Screw_Terminal_01x01
- added J7: Iout, TerminalBlock_MetzConnect:TerminalBlock_MetzConnect_360271_1x01_Horizontal_ScrewM3.0_Boxed, symbol Connector:Screw_Terminal_01x01
- added J8: IN, TerminalBlock_MetzConnect:TerminalBlock_MetzConnect_360271_1x01_Horizontal_ScrewM3.0_Boxed, symbol Connector:Screw_Terminal_01x01
- added KEY1: menu, K2-1103DT-A4CW-04:KEY-TH_4P-L12.0-W12.0-P5.00-LS13.4, symbol K2-1103DT-A4CW-04:K2-1103DT-A4CW-04
- added KEY2: select, K2-1103DT-A4CW-04:KEY-TH_4P-L12.0-W12.0-P5.00-LS13.4, symbol K2-1103DT-A4CW-04:K2-1103DT-A4CW-04
- added PS1: HLK-PM01, Converter_ACDC:Converter_ACDC_HiLink_HLK-PMxx, symbol Converter_ACDC:HLK-PM01
- added Q1: BTA16-600B, Package_TO_SOT_THT:TO-220-3_Vertical, symbol Triac_Thyristor:BTA16-600B
- added R5: 1K, Resistor_THT:R_Axial_DIN0207_L6.3mm_D2.5mm_P10.16mm_Horizontal, symbol Device:R
- added R8: Heater, TerminalBlock:TerminalBlock_bornier-2_P5.08mm, symbol Device:Heater
- added RV1: 5K, Potentiometer_THT:Potentiometer_Alps_RK09Y11_Single_Horizontal, symbol Device:R_Potentiometer
- added U2: HS96L03W2C03, OLEDTHL27:OLED-TH_L27.8-W27.2-P2.54_C9900033791, symbol OLEDTTHL27:HS96L03W2C03
- added U3: PC817, Package_DIP:DIP-4_W7.62mm, symbol Isolator:PC817
- added U4: MOC3010, TFGMOC:DIP-6_L9.6-W6.4-P2.54-LS7.6-BL, symbol TFGMOC:MOC3010
- BZ1: footprint Buzzer_Beeper:Buzzer_12x9.5RM7.6 -> digikey-footprints:Piezo_Transducer_THT_PS1240P02BT
- H3, H4: value MountingHole -> MH; footprint MountingHole:MountingHole_3.2mm_M3_Pad_Via -> MountingHole:MountingHole_3mm_Pad_Via
- R1: value 10K -> 1K; footprint Resistor_SMD:R_1206_3216Metric -> Resistor_THT:R_Axial_DIN0207_L6.3mm_D2.5mm_P10.16mm_Horizontal
- R2: value 10k -> 1K; footprint Resistor_SMD:R_1206_3216Metric -> Resistor_THT:R_Axial_DIN0207_L6.3mm_D2.5mm_P10.16mm_Horizontal
- R3, R4: value 10k -> 47K; footprint Resistor_SMD:R_1206_3216Metric -> Resistor_THT:R_Axial_DIN0207_L6.3mm_D2.5mm_P10.16mm_Horizontal
- R6: value 100k -> 220; footprint Resistor_SMD:R_1206_3216Metric -> Resistor_THT:R_Axial_DIN0207_L6.3mm_D2.5mm_P10.16mm_Horizontal
- R7: value 22k -> 100; footprint Resistor_SMD:R_1206_3216Metric -> Resistor_THT:R_Axial_DIN0207_L6.3mm_D2.5mm_P10.16mm_Horizontal
- U1: footprint ESP32-DEVKIT-V1:MODULE_ESP32_DEVKIT_V1 -> esp32devkitv1:MODULE_ESP32_DEVKIT_V1; Availability (none) -> Not in stock; Check_prices (none) -> https://www.snapeda.com/parts/ESP32-DEVKIT-V1/Do+it/view-pa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; MF (none) -> Do it; MP (none) -> ESP32-DEVKIT-V1; Package (none) -> None; Price (none) -> None; SnapEDA_Link (none) -> https://www.snapeda.com/parts/ESP32-DEVKIT-V1/Do+it/view-pa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
Connections:
- net +5V: now also PS1.4 (+Vout)
- net GND: now also R1.2, R2.2, J4.5 (Pin_5), PS1.3 (-Vout), R5.1, RV1.1, U2.1 (GND), U4.2; no longer R1.1, R2.1, R3.1, R4.1
- net GPIO 4: now also R7.2; no longer R1.2
- net SDA: now also U2.4 (SDA)
- net SOUND: now also U1.20 (D35)
- net at R6.2: now also U4.6
- net at R7.1: now also U4.1
- net GPIO 19: now reaches U1.10 (D19)
- net GPIO 19: now also R5.2, U3.3
- net SO: now reaches U1.15 (D23)
- net SO: now also J4.1 (Pin_1)
- net SCK: now reaches U1.9 (D18)
- net SCK: now also J4.3 (Pin_3)
- net +3V3 renamed 3v3
- net 3v3: now also J4.4 (Pin_4), KEY1.4, KEY2.4, RV1.3, U2.2 (VCC), U3.4
- net GPIO 12: no longer names the net of R3.2
- net GPIO 12: now also D1.4; no longer U1.27 (D12)
- net GPIO 13: no longer names the net of U1.28 (D13)
- net GPIO 13: no longer R4.2
- net GPIO 14: no longer names the net of U1.26 (D14)
- net GPIO 5 renamed CS
- net CS: now also J4.2 (Pin_2); no longer R2.2
- net MOTOR A1 renamed GPIO 27
- net GPIO 27: now also RV1.2
- net MOTOR A2: no longer names the net of U1.24 (D26)
- net MOTOR B1 renamed GPIO 33
- net GPIO 33: now also R2.1, KEY2.2
- net MOTOR B2 renamed GPIO 32
- net GPIO 32: now also R1.1, KEY1.2
- net SCL renamed SLC
- net SLC: now also U2.3 (SCL)
- net TCK B renamed L
- net L: now also R3.1, F3.1, J7.1 (Pin_1), Q1.2 (A2)
- new net: F3.2, PS1.1 (AC/L)
- new net: D1.2, R4.1
- new net: F1.2, J6.1 (Pin_1)
- new net: D1.1 (+), U3.1
- new net: D1.3 (-), U3.2
- new net: Q1.3 (G), U4.4
- new net: Q1.1 (A1), R8.1
- new net: F1.1, J5.1 (Pin_1)
- new net N: J2.1 (Pin_1), J8.1 (Pin_1), PS1.2 (AC/N), R4.2, R8.2
- no-connect marks 15 -> 21
Other:
- note added: "AC Power Supply: 120Vrms"
- note added: "DC Power Supply: 5V"
- note added: "ESP32 Module: Controller"
- note added: "Feedback"
- note added: "Final Control Element: Thyristor"
- note added: "UI Indicator: OLED & Buzzer"
- note added: "UI Interactions: Btn & Pot"
- note added: "Zero Crossing"
- note removed: "AC POWER SUPPLY"
- note removed: "ESP 32 MODULE"
- note removed: "ESP 32 POWER"
- note removed: "FEEDBACK"
- note removed: "FINAL CONTROL ELEMENT"
- note removed: "SCREWS"
- note removed: "UI INDICATORS"
- note removed: "UI INTERFACE"

Commit message: PCB view
Other:
- company: (none) -> ET
- title: Thermo Forge 53  -> ThermoForge TFG-ET V1
Changed lines of the file:
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@@
   (paper "A4")
   (title_block
-    (title "Thermo Forge 53 ")
+    (title "ThermoForge TFG-ET V1")
+    (date "2024-11-29")
+    (company "ET")
   )
   (junction (at 153.67 45.72) (diameter 0) (color 0 0 0 0)
